File: mcu_datalogger.kicad_pcb (KiCad board)
At the start: 2 copper layers, 29 parts, among them J1 Conn_01x04_Pin, J2 Conn_01x04_Pin, J3 Conn_01x09, J4 Conn_02x03_Counter_Clockwise, U1 DS1337S_, U3 24LC1025, U4 24LC1025, U5 ATMEGA328P-AU, Y1 32.768 KHz, Y2 16MHz

Commit message: PCB Layout Started
Parts:
- moved H2 116.8 mm to (227.4, 66.7)
- moved H4 114.4 mm to (227.4, 92.0)
- moved U5 83.5 mm to (205.8, 75.1)
- moved J4 79.5 mm to (225.3, 71.2)
- moved J1 77.2 mm to (227.9, 79.9)
- moved U1 71.8 mm to (192.9, 86.8)
- moved H1 71.6 mm to (182.1, 66.7)
- moved Y2 70.0 mm to (205.9, 83.5)
- moved H3 68.8 mm to (182.1, 91.9)
- moved U3 68.5 mm to (192.7, 72.1)
- moved U4 68.4 mm to (192.7, 79.4)
- moved J2 56.9 mm to (212.4, 91.9), turned to 90 degrees
- moved Y1 48.9 mm to (185.3, 84.8), turned to 90 degrees
- moved J3 40.7 mm to (186.9, 91.9), turned to 90 degrees
Other:
- board outline added: 50 x 30 mm

Commit message: Layout almost completed
Parts:
- moved R3 102.2 mm to (219.2, 73.1)
- moved R1 101.6 mm to (219.1, 70.1)
- moved R5 98.9 mm to (215.1, 75.9), turned to 180 degrees
- moved R4 98.8 mm to (215.0, 73.1), turned to 180 degrees
- moved R2 98.0 mm to (214.9, 70.1), turned to 180 degrees
- moved D1 87.0 mm to (219.1, 67.1)
- moved D2 84.5 mm to (214.8, 67.1)
- moved C4 84.2 mm to (215.2, 82.0), turned to 180 degrees
- moved C3 84.1 mm to (215.2, 79.3), turned to 180 degrees
- moved BT2 80.6 mm to (185.0, 73.6)
- moved C2 78.8 mm to (205.4, 66.8)
- moved C5 77.4 mm to (209.8, 66.8)
- moved R6 77.3 mm to (194.8, 87.4), turned to 180 degrees
- moved R7 74.1 mm to (191.0, 87.4)
- moved C1 73.6 mm to (201.2, 66.8)
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Connections:
- D2 pad 2: /SCK -> Net-(BT2-+)
- J4 pad 2: /SCK -> /Vcc
- J4 pad 3: /RESET -> /SCK
- J4 pad 4: GND -> /MOSI
- J4 pad 5: /MOSI -> /RESET
Routing:
- net /Vcc: track 0.00 -> 95.0 mm, vias 0 -> 1
- net /SCK: track 0.00 -> 70.4 mm, vias 0 -> 2
- net Net-(BT2-+): track 0.00 -> 62.1 mm, vias 0 -> 4
- net /SDA: track 0.00 -> 58.1 mm, vias 0 -> 2
- net GND: track 0.00 -> 49.2 mm, vias 0 -> 5
- net /TX: track 0.00 -> 28.5 mm, vias 0 -> 1
- net /D2: track 0.00 -> 27.3 mm, vias 0 -> 1
- net /D3: track 0.00 -> 26.9 mm
- net /RX: track 0.00 -> 25.4 mm, vias 0 -> 1
- net /D4: track 0.00 -> 24.3 mm
- net Net-(U5-PB6): track 0.00 -> 23.3 mm, vias 0 -> 2
- net /RESET: track 0.00 -> 23.2 mm, vias 0 -> 4
- net /MOSI: track 0.00 -> 22.5 mm
- net Net-(U5-PB7): track 0.00 -> 18.8 mm
- net /MISO: track 0.00 -> 18.3 mm, vias 0 -> 1
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Other:
- board size 50 x 30 mm -> 50.6 x 30.6 mm
